File: Populated_PLG_sensor.sch (EAGLE design)
At the start: 21 parts, among them CON1 USB_MOLEX_0480372200, J1 MICRO-SD_CARD_SOCKET, SW1 SPST_TACT-KMR2, SW2 SPST_TACT-KMR2, SW3 SPST_TACT-KMR2, SW4 SPST_TACT-KMR2

Commit message: Updated layout
Incomplete, uploading for Rob to look at
Connections:
- removed net N$12: R9.1, SW2.S, SW2.S1
- removed net N$15: R8.1, SW4.S, SW4.S1
- removed net N$7: R7.1, X2.RESET
- new net MASTER_RST: R9.1, SW2.S, X1.RESET
- new net SLAVE_RST: R7.1, R8.1, SW4.S, X2.RESET
- new net SLV_GND: R6.2, X2.GND
- net GND: no longer R6.2, SW1.S1, SW2.P1, SW3.S1, SW4.P1, X2.GND
- net MASTER_GPIO0: no longer SW1.P1
- net SLAVE_GPIO0: no longer SW3.P1
Other:
- moved on the sheet: R7
Changed lines of the file:
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@@
 <part name="SUPPLY7" library="SparkFun-PowerSymbols" deviceset="VIN" device=""/>
 <part name="GND5" library="SparkFun-PowerSymbols" deviceset="GND" device=""/>
-<part name="GND6" library="SparkFun-PowerSymbols" deviceset="GND" device=""/>
-<part name="GND7" library="SparkFun-PowerSymbols" deviceset="GND" device=""/>
 <part name="SUPPLY8" library="SparkFun-PowerSymbols" deviceset="3.3V" device=""/>
 <part name="SUPPLY9" library="SparkFun-PowerSymbols" deviceset="3.3V" device=""/>
@@
 <instance part="SUPPLY2" gate="G$1" x="220.98" y="129.54" rot="R270"/>
 <instance part="GND1" gate="1" x="195.58" y="91.44"/>
-<instance part="GND2" gate="1" x="137.16" y="83.82"/>
-<instance part="GND3" gate="1" x="137.16" y="132.08"/>
+<instance part="GND2" gate="1" x="137.16" y="81.28"/>
+<instance part="GND3" gate="1" x="137.16" y="129.54"/>
 <instance part="GND4" gate="1" x="220.98" y="121.92"/>
 <instance part="SUPPLY3" gate="G$1" x="190.5" y="68.58"/>
@@
 <instance part="SUPPLY7" gate="G$1" x="220.98" y="134.62"/>
 <instance part="GND5" gate="1" x="210.82" y="40.64"/>
-<instance part="GND6" gate="1" x="149.86" y="132.08"/>
-<instance part="GND7" gate="1" x="149.86" y="83.82"/>
 <instance part="SUPPLY8" gate="G$1" x="154.94" y="142.24" rot="R270"/>
 <instance part="SUPPLY9" gate="G$1" x="83.82" y="149.86" rot="R90"/>
@@
 <instance part="SUPPLY12" gate="G$1" x="38.1" y="104.14" rot="R90"/>
 <instance part="SUPPLY13" gate="G$1" x="38.1" y="152.4" rot="R90"/>
-<instance part="R7" gate="G$1" x="91.44" y="109.22" rot="R180"/>
+<instance part="R7" gate="G$1" x="91.44" y="114.3" rot="R180"/>
 <instance part="SW1" gate="G$1" x="45.72" y="48.26" rot="R270"/>
 <instance part="SW2" gate="G$1" x="35.56" y="27.94" rot="R270"/>
@@
 <net name="GND" class="0">
 <segment>
-<pinref part="R1" gate="G$1" pin="2"/>
-<pinref part="GND6" gate="1" pin="GND"/>
-<wire x1="147.32" y1="137.16" x2="149.86" y2="134.62" width="0.1524" layer="91"/>
-</segment>
-<segment>
-<pinref part="R6" gate="G$1" pin="2"/>
-<pinref part="GND7" gate="1" pin="GND"/>
-<wire x1="149.86" y1="86.36" x2="147.32" y2="88.9" width="0.1524" layer="91"/>
-</segment>
-<segment>
 <pinref part="GND5" gate="1" pin="GND"/>
 <pinref part="J1" gate="1" pin="GND"/>
@@
 </segment>
 <segment>
-<pinref part="X2" gate="G$1" pin="GND"/>
-<pinref part="GND2" gate="1" pin="GND"/>
-<wire x1="134.62" y1="88.9" x2="137.16" y2="86.36" width="0.1524" layer="91"/>
-</segment>
-<segment>
 <pinref part="U$1" gate="G$1" pin="GND"/>
 <pinref part="GND4" gate="1" pin="GND"/>
@@
 </segment>
 <segment>
-<pinref part="X1" gate="G$1" pin="GND"/>
-<pinref part="GND3" gate="1" pin="GND"/>
-<wire x1="134.62" y1="137.16" x2="137.16" y2="134.62" width="0.1524" layer="91"/>
-</segment>
-<segment>
-<pinref part="SW1" gate="G$1" pin="S1"/>
 <pinref part="SW1" gate="G$1" pin="S"/>
-<wire x1="50.8" y1="45.72" x2="50.8" y2="48.26" width="0.1524" layer="91"/>
-<junction x="50.8" y="48.26"/>
 <pinref part="GND12" gate="1" pin="GND"/>
 <wire x1="50.8" y1="48.26" x2="55.88" y2="48.26" width="0.1524" layer="91"/>
@@
 </segment>
 <segment>
-<pinref part="SW3" gate="G$1" pin="S1"/>
 <pinref part="SW3" gate="G$1" pin="S"/>
-<wire x1="114.3" y1="45.72" x2="114.3" y2="48.26" width="0.1524" layer="91"/>
-<junction x="114.3" y="48.26"/>
 <pinref part="GND13" gate="1" pin="GND"/>
 <wire x1="114.3" y1="48.26" x2="119.38" y2="48.26" width="0.1524" layer="91"/>
@@
 </segment>
 <segment>
-<pinref part="SW4" gate="G$1" pin="P1"/>
 <pinref part="SW4" gate="G$1" pin="P"/>
-<wire x1="93.98" y1="25.4" x2="93.98" y2="27.94" width="0.1524" layer="91"/>
 <wire x1="93.98" y1="27.94" x2="91.44" y2="27.94" width="0.1524" layer="91"/>
-<junction x="93.98" y="27.94"/>
 <pinref part="GND11" gate="1" pin="GND"/>
 <wire x1="91.44" y1="27.94" x2="88.9" y2="25.4" width="0.1524" layer="91"/>
 </segment>
 <segment>
-<pinref part="SW2" gate="G$1" pin="P1"/>
 <pinref part="SW2" gate="G$1" pin="P"/>
-<wire x1="30.48" y1="25.4" x2="30.48" y2="27.94" width="0.1524" layer="91"/>
 <wire x1="30.48" y1="27.94" x2="27.94" y2="27.94" width="0.1524" layer="91"/>
-<junction x="30.48" y="27.94"/>
 <pinref part="GND10" gate="1" pin="GND"/>
 <wire x1="27.94" y1="27.94" x2="25.4" y2="25.4" width="0.1524" layer="91"/>
+</segment>
+<segment>
+<pinref part="R1" gate="G$1" pin="2"/>
+<wire x1="147.32" y1="137.16" x2="147.32" y2="134.62" width="0.1524" layer="91"/>
+<wire x1="147.32" y1="134.62" x2="144.78" y2="132.08" width="0.1524" layer="91"/>
+<pinref part="GND3" gate="1" pin="GND"/>
+<wire x1="144.78" y1="132.08" x2="137.16" y2="132.08" width="0.1524" layer="91"/>
+<pinref part="X1" gate="G$1" pin="GND"/>
+<wire x1="134.62" y1="137.16" x2="134.62" y2="134.62" width="0.1524" layer="91"/>
+<wire x1="134.62" y1="134.62" x2="137.16" y2="132.08" width="0.1524" layer="91"/>
+<junction x="137.16" y="132.08"/>
 </segment>
 </net>
@@
 </segment>
 </net>
-<net name="N$7" class="0">
-<segment>
-<pinref part="X2" gate="G$1" pin="RESET"/>
-<pinref part="R7" gate="G$1" pin="1"/>
-<wire x1="99.06" y1="106.68" x2="96.52" y2="109.22" width="0.1524" layer="91"/>
-</segment>
-</net>
 <net name="ESP_RST" class="0">
 <segment>
 <pinref part="R7" gate="G$1" pin="2"/>
-<wire x1="86.36" y1="109.22" x2="83.82" y2="109.22" width="0.1524" layer="91"/>
-<label x="83.82" y="109.22" size="1.27" layer="95" rot="R180" xref="yes"/>
+<wire x1="86.36" y1="114.3" x2="83.82" y2="114.3" width="0.1524" layer="91"/>
+<label x="83.82" y="114.3" size="1.27" layer="95" rot="R180" xref="yes"/>
 </segment>
 <segment>
@@
 </segment>
 </net>
-<net name="N$12" class="0">
-<segment>
-<pinref part="SW2" gate="G$1" pin="S"/>
-<pinref part="SW2" gate="G$1" pin="S1"/>
-<wire x1="40.64" y1="27.94" x2="40.64" y2="25.4" width="0.1524" layer="91"/>
-<junction x="40.64" y="27.94"/>
-<pinref part="R9" gate="G$1" pin="1"/>
-<wire x1="40.64" y1="27.94" x2="45.72" y2="27.94" width="0.1524" layer="91"/>
-</segment>
-</net>
-<net name="N$15" class="0">
-<segment>
-<pinref part="SW4" gate="G$1" pin="S1"/>
-<pinref part="SW4" gate="G$1" pin="S"/>
-<wire x1="104.14" y1="25.4" x2="104.14" y2="27.94" width="0.1524" layer="91"/>
-<junction x="104.14" y="27.94"/>
-<pinref part="R8" gate="G$1" pin="1"/>
-<wire x1="109.22" y1="27.94" x2="104.14" y2="27.94" width="0.1524" layer="91"/>
-</segment>
-</net>
 <net name="MASTER_GPIO0" class="0">
 <segment>
@@
 </segment>
 <segment>
-<pinref part="SW1" gate="G$1" pin="P1"/>
 <pinref part="SW1" gate="G$1" pin="P"/>
-<wire x1="40.64" y1="45.72" x2="40.64" y2="48.26" width="0.1524" layer="91"/>
 <wire x1="40.64" y1="48.26" x2="38.1" y2="48.26" width="0.1524" layer="91"/>
-<junction x="40.64" y="48.26"/>
 <label x="38.1" y="48.26" size="1.27" layer="95" rot="R180" xref="yes"/>
 </segment>
@@
 <segment>
 <pinref part="SW3" gate="G$1" pin="P"/>
-<pinref part="SW3" gate="G$1" pin="P1"/>
-<wire x1="104.14" y1="48.26" x2="104.14" y2="45.72" width="0.1524" layer="91"/>
 <wire x1="104.14" y1="48.26" x2="101.6" y2="48.26" width="0.1524" layer="91"/>
-<junction x="104.14" y="48.26"/>
 <label x="101.6" y="48.26" size="1.27" layer="95" rot="R180" xref="yes"/>
 </segment>
@@
 </segment>
 </net>
-<net name="N$5" class="0">
+<net name="N$8" class="0">
 <segment>
 <pinref part="X2" gate="G$1" pin="GPIO15"/>
@@
 </segment>
 </net>
+<net name="SLV_GND" class="0">
+<segment>
+<pinref part="X2" gate="G$1" pin="GND"/>
+<pinref part="GND2" gate="1" pin="GND"/>
+<wire x1="134.62" y1="88.9" x2="134.62" y2="86.36" width="0.1524" layer="91"/>
+<wire x1="134.62" y1="86.36" x2="137.16" y2="83.82" width="0.1524" layer="91"/>
+<pinref part="R6" gate="G$1" pin="2"/>
+<wire x1="147.32" y1="88.9" x2="147.32" y2="86.36" width="0.1524" layer="91"/>
+<wire x1="147.32" y1="86.36" x2="144.78" y2="83.82" width="0.1524" layer="91"/>
+<wire x1="144.78" y1="83.82" x2="137.16" y2="83.82" width="0.1524" layer="91"/>
+<junction x="137.16" y="83.82"/>
+</segment>
+</net>
+<net name="SLAVE_RST" class="0">
+<segment>
+<pinref part="X2" gate="G$1" pin="RESET"/>
+<pinref part="R7" gate="G$1" pin="1"/>
+<wire x1="99.06" y1="106.68" x2="99.06" y2="111.76" width="0.1524" layer="91"/>
+<wire x1="99.06" y1="111.76" x2="96.52" y2="114.3" width="0.1524" layer="91"/>
+<wire x1="99.06" y1="106.68" x2="96.52" y2="106.68" width="0.1524" layer="91"/>
+<wire x1="96.52" y1="106.68" x2="93.98" y2="109.22" width="0.1524" layer="91"/>
+<junction x="99.06" y="106.68"/>
+<label x="93.98" y="109.22" size="1.4224" layer="95" rot="R180" xref="yes"/>
+</segment>
+<segment>
+<pinref part="SW4" gate="G$1" pin="S"/>
+<pinref part="R8" gate="G$1" pin="1"/>
+<wire x1="109.22" y1="27.94" x2="104.14" y2="27.94" width="0.1524" layer="91"/>
+<wire x1="109.22" y1="27.94" x2="109.22" y2="25.4" width="0.1524" layer="91"/>
+<wire x1="109.22" y1="25.4" x2="106.68" y2="22.86" width="0.1524" layer="91"/>
+<junction x="109.22" y="27.94"/>
+<label x="106.68" y="22.86" size="1.4224" layer="95" rot="R180" xref="yes"/>
+</segment>
+</net>
+<net name="MASTER_RST" class="0">
+<segment>
+<pinref part="X1" gate="G$1" pin="RESET"/>
+<wire x1="99.06" y1="154.94" x2="96.52" y2="157.48" width="0.1524" layer="91"/>
+<label x="96.52" y="157.48" size="1.4224" layer="95" rot="R180" xref="yes"/>
+</segment>
+<segment>
+<pinref part="SW2" gate="G$1" pin="S"/>
+<pinref part="R9" gate="G$1" pin="1"/>
+<wire x1="40.64" y1="27.94" x2="45.72" y2="27.94" width="0.1524" layer="91"/>
+<wire x1="45.72" y1="27.94" x2="45.72" y2="25.4" width="0.1524" layer="91"/>
+<wire x1="45.72" y1="25.4" x2="43.18" y2="22.86" width="0.1524" layer="91"/>
+<junction x="45.72" y="27.94"/>
+<label x="43.18" y="22.86" size="1.4224" layer="95" rot="R180" xref="yes"/>
+</segment>
+</net>

Commit message: Improved
Parts:
- added C1, C2: 10uF, SparkFun-Capacitors:10UF-0603-6.3V-20%
- added CON2: 4_PIN_HEADER, Other:4_PIN_HEADER
Connections:
- removed net N$3: R2.1, X1.GPIO2
- removed net N$6: R5.1, X2.GPIO2
- removed net SLV_GND: R6.2, X2.GND
- new net MASTER_DEBUG: CON2.S_DBG, R2.1, X1.GPIO2
- new net SLAVE_DEBUG: CON2.M_DBG, R5.1, X2.GPIO2
- net GND: now also C1.2, C2.2, CON2.GND, CON2.GND2, R6.2, X2.GND
- net VIN: now also C1.1, C2.1
Other:
- moved on the sheet: R2, R5
